File: kicad_src/hv-isol-meas.kicad_pcb (KiCad board)
At the start: 2 copper layers, 98.8 x 48.9 mm, 62 parts, among them J1 MEAS_OUT, J2 PSU_IN, J3 DC-Socket, U1 OPA2197DGK, U2 MCP1541-TT, U3 OPA197xDBV, U4 DC-DC-SIP-DUAL-ISOL, U5 MCP1541T, U6 TPS60403

Commit message: Add files via upload
Parts:
- removed R16, R9: 1k, Resistor_SMD:R_0805_2012Metric_Pad1.20x1.40mm_HandSolder
- removed REF** (x2): Symbol_Highvoltage_Type1_CopperTop_Small, Symbol:Symbol_Highvoltage_Type1_CopperTop_Small
- removed REF**: Symbol_Barrel_Polarity, Symbol:Symbol_Barrel_Polarity
- added C20: 1u, Capacitor_SMD:C_0805_2012Metric_Pad1.18x1.45mm_HandSolder, F.Cu at (63.2, 111.1)
- added FB1: FB_0805, Resistor_SMD:R_0805_2012Metric_Pad1.20x1.40mm_HandSolder, F.Cu at (109.2, 120.0)
- added FB2: FB_0805, Resistor_SMD:R_0805_2012Metric_Pad1.20x1.40mm_HandSolder, F.Cu at (82.5, 100.3)
- R2: value 47k -> 0R
Routing:
- net Net-(U6-IN): track 5.48 -> 7.58 mm
Other:
- board text added: "Rev 1.1"
- board text removed: "Rev 1.0"
