File: kicad_src/hv-isol-meas.kicad_sch (KiCad schematic)
At the start: 59 parts, among them J1 MEAS_OUT, J2 PSU_IN, J3 DC-Socket, U1 OPA2197DGK, U2 MCP1541-TT, U3 OPA197xDBV, U4 DC-DC-SIP-DUAL-ISOL, U5 MCP1541T, U6 TPS60403

Commit message: Add files via upload
Parts:
- removed R16, R9: 1k, Resistor_SMD:R_0805_2012Metric_Pad1.20x1.40mm_HandSolder, symbol Device:R
- added C20: 1u, Capacitor_SMD:C_0805_2012Metric_Pad1.18x1.45mm_HandSolder, symbol Device:C_Small
- added FB1, FB2: FB_0805, Resistor_SMD:R_0805_2012Metric_Pad1.20x1.40mm_HandSolder, symbol Device:FerriteBead_Small
- R2: value 47k -> 0R
Connections:
- net +VREF: now also FB2.2
- net +VREFA: now also FB1.2
- net 0V: now also C20.2
- net at C14.1, U5.2 (Vout): now also FB2.1
- net at L5.4, U6.2 (IN): now also C20.1
- net at C4.1, U2.2 (Vout): now also FB1.1
Other:
- note added: "1.1"
- note removed: "1"
Changed lines of the file:
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@@
   (junction (at 200.66 101.6) (diameter 0) (color 0 0 0 0)
+  )
+  (junction (at 53.34 139.7) (diameter 0) (color 0 0 0 0)
   )
   (junction (at 152.4 45.72) (diameter 0) (color 0 0 0 0)
@@
     (stroke (width 0) (type default))
   )
-  (wire (pts (xy 142.24 80.01) (xy 143.51 80.01))
+  (wire (pts (xy 142.24 80.01) (xy 144.78 80.01))
     (stroke (width 0) (type default))
   )
@@
     (stroke (width 0) (type dash))
   )
-  (wire (pts (xy 142.24 114.3) (xy 143.51 114.3))
+  (wire (pts (xy 142.24 114.3) (xy 144.78 114.3))
     (stroke (width 0) (type default))
   )
@@
     (stroke (width 0) (type default))
   )
-  (wire (pts (xy 151.13 114.3) (xy 153.67 114.3))
-    (stroke (width 0) (type default))
-  )
   (wire (pts (xy 240.03 54.61) (xy 234.95 54.61))
     (stroke (width 0) (type default))
@@
     (stroke (width 0) (type default))
   )
+  (wire (pts (xy 149.86 114.3) (xy 153.67 114.3))
+    (stroke (width 0) (type default))
+  )
   (wire (pts (xy 116.84 72.39) (xy 116.84 77.47))
     (stroke (width 0) (type default))
@@
     (stroke (width 0) (type default))
   )
-  (wire (pts (xy 153.67 80.01) (xy 151.13 80.01))
+  (wire (pts (xy 149.86 80.01) (xy 153.67 80.01))
     (stroke (width 0) (type default))
   )
@@
     (effects (font (size 1.27 1.27)) (justify left bottom))
   )
-  (text "1" (at 270.51 194.31 0)
+  (text "1.1" (at 270.51 194.31 0)
     (effects (font (size 3 3)) (justify left bottom))
   )
@@
     )
   )
-  (symbol (lib_id "Device:R") (at 147.32 114.3 90) (unit 1)
-    (in_bom yes) (on_board yes) (dnp no)
-    (property "Reference" "R9" (at 147.32 109.22 90)
-      (effects (font (size 1.27 1.27)))
-    )
-    (property "Value" "1k" (at 147.32 111.76 90)
-      (effects (font (size 1.27 1.27)))
-    )
-    (property "Footprint" "Resistor_SMD:R_0805_2012Metric_Pad1.20x1.40mm_HandSolder" (at 147.32 116.078 90)
-      (effects (font (size 1.27 1.27)) hide)
-    )
-    (property "Datasheet" "~" (at 147.32 114.3 0)
-      (effects (font (size 1.27 1.27)) hide)
-    )
-    (pin "1")
-    (pin "2")
-    (instances
-      (project "hv-isol-meas"
-        (path "/f5fb5782-757d-4f04-9fc4-3ef5f648ef9f"
-          (reference "R9") (unit 1)
+  (symbol (lib_id "User_Global_Symbol_Library:0V") (at 53.34 144.78 0) (unit 1)
+    (in_bom yes) (on_board yes) (dnp no)
+    (property "Reference" "#PWR049" (at 53.34 149.86 0)
+      (effects (font (size 1.27 1.27)) hide)
+    )
+    (property "Value" "0V" (at 53.34 147.32 0)
+      (effects (font (size 1.27 1.27)))
+    )
+    (property "Footprint" "" (at 53.34 144.78 0)
+      (effects (font (size 1.27 1.27)) hide)
+    )
+    (property "Datasheet" "" (at 53.34 144.78 0)
+      (effects (font (size 1.27 1.27)) hide)
+    )
+    (pin "1")
+    (instances
+      (project "hv-isol-meas"
+        (path "/f5fb5782-757d-4f04-9fc4-3ef5f648ef9f"
+          (reference "#PWR049") (unit 1)
         )
       )
@@
         (path "/f5fb5782-757d-4f04-9fc4-3ef5f648ef9f"
           (reference "#PWR021") (unit 1)
+        )
+      )
+    )
+  )
+  (symbol (lib_id "Device:C_Small") (at 53.34 142.24 0) (mirror y) (unit 1)
+    (in_bom yes) (on_board yes) (dnp no)
+    (property "Reference" "C20" (at 49.53 142.24 0)
+      (effects (font (size 1.27 1.27)))
+    )
+    (property "Value" "1u" (at 49.53 144.78 0)
+      (effects (font (size 1.27 1.27)))
+    )
+    (property "Footprint" "Capacitor_SMD:C_0805_2012Metric_Pad1.18x1.45mm_HandSolder" (at 53.34 142.24 0)
+      (effects (font (size 1.27 1.27)) hide)
+    )
+    (property "Datasheet" "~" (at 53.34 142.24 0)
+      (effects (font (size 1.27 1.27)) hide)
+    )
+    (pin "1")
+    (pin "2")
+    (instances
+      (project "hv-isol-meas"
+        (path "/f5fb5782-757d-4f04-9fc4-3ef5f648ef9f"
+          (reference "C20") (unit 1)
         )
       )
@@
     )
   )
+  (symbol (lib_id "Device:FerriteBead_Small") (at 147.32 80.01 90) (unit 1)
+    (in_bom yes) (on_board yes) (dnp no) (fields_autoplaced)
+    (property "Reference" "FB1" (at 147.2819 73.66 90)
+      (effects (font (size 1.27 1.27)))
+    )
+    (property "Value" "FB_0805" (at 147.2819 76.2 90)
+      (effects (font (size 1.27 1.27)))
+    )
+    (property "Footprint" "Resistor_SMD:R_0805_2012Metric_Pad1.20x1.40mm_HandSolder" (at 147.32 81.788 90)
+      (effects (font (size 1.27 1.27)) hide)
+    )
+    (property "Datasheet" "~" (at 147.32 80.01 0)
+      (effects (font (size 1.27 1.27)) hide)
+    )
+    (pin "1")
+    (pin "2")
+    (instances
+      (project "hv-isol-meas"
+        (path "/f5fb5782-757d-4f04-9fc4-3ef5f648ef9f"
+          (reference "FB1") (unit 1)
+        )
+      )
+    )
+  )
+  (symbol (lib_id "Device:FerriteBead_Small") (at 147.32 114.3 90) (unit 1)
+    (in_bom yes) (on_board yes) (dnp no) (fields_autoplaced)
+    (property "Reference" "FB2" (at 147.2819 107.95 90)
+      (effects (font (size 1.27 1.27)))
+    )
+    (property "Value" "FB_0805" (at 147.2819 110.49 90)
+      (effects (font (size 1.27 1.27)))
+    )
+    (property "Footprint" "Resistor_SMD:R_0805_2012Metric_Pad1.20x1.40mm_HandSolder" (at 147.32 116.078 90)
+      (effects (font (size 1.27 1.27)) hide)
+    )
+    (property "Datasheet" "~" (at 147.32 114.3 0)
+      (effects (font (size 1.27 1.27)) hide)
+    )
+    (pin "1")
+    (pin "2")
+    (instances
+      (project "hv-isol-meas"
+        (path "/f5fb5782-757d-4f04-9fc4-3ef5f648ef9f"
+          (reference "FB2") (unit 1)
+        )
+      )
+    )
+  )
   (symbol (lib_id "Device:R") (at 195.58 128.27 90) (mirror x) (unit 1)
     (in_bom yes) (on_board yes) (dnp no)
@@
       (effects (font (size 1.27 1.27)))
     )
-    (property "Value" "47k" (at 208.28 49.53 90)
+    (property "Value" "0R" (at 208.28 49.53 90)
       (effects (font (size 1.27 1.27)))
     )
@@
         )
       )
-    )
-  )
-  (symbol (lib_id "Device:R") (at 147.32 80.01 90) (unit 1)
-    (in_bom yes) (on_board yes) (dnp no)
-    (property "Reference" "R16" (at 147.32 74.93 90)
-      (effects (font (size 1.27 1.27)))
-    )
-    (property "Value" "1k" (at 147.32 77.47 90)
-      (effects (font (size 1.27 1.27)))
-    )
-    (property "Footprint" "Resistor_SMD:R_0805_2012Metric_Pad1.20x1.40mm_HandSolder" (at 147.32 81.788 90)
-      (effects (font (size 1.27 1.27)) hide)
-    )
-    (property "Datasheet" "~" (at 147.32 80.01 0)
-      (effects (font (size 1.27 1.27)) hide)
-    )
-    (pin "1")
-    (pin "2")
-    (instances
-      (project "hv-isol-meas"
-        (path "/f5fb5782-757d-4f04-9fc4-3ef5f648ef9f"
-          (reference "R16") (unit 1)
-        )
-      )
